Commit message: update

File: gazebo_ros_demos/rrbot_description/urdf/rrbot.xacro (robot description, xacro)
@@ -15,10 +15,20 @@
   <xacro:property name="height6"   value="0.125" /> <!-- Link 6 -->
   <xacro:property name="heightEEF" value="0.03" /> <!-- Link 7  EEF Link-->
-  <xacro:property name="MinAngle"  value="-2.24346" /> <!-- Min angle-->
-  <xacro:property name="MaxAngle"  value="2.24346" /> <!-- Max angle-->
+  <!-- upper limit of the angle -->
+  <xacro:property name="UpperLim_roll"  value="2.617" />
+  <xacro:property name="UpperLim_joint1"  value="1.46239" />
+  <xacro:property name="UpperLim_joint3"  value="2.26006" />
+  <xacro:property name="UpperLim_joint5"  value="1.958382" />
+  <xacro:property name="LowerLim_roll"  value= "-2.617" />
+  <xacro:property name="LowerLim_joint1"  value="-1.8816" />
+  <xacro:property name="LowerLim_joint3"  value="-1.7385" />
+  <xacro:property name="LowerLim_joint5"  value="-1.677152" />
   <xacro:property name="heightEEF" value="0.03" /> <!-- Link 7  EEF Link-->
   <xacro:property name="damp_value"  value="0.0" /> <!-- Link 6 -->
-  <xacro:property name="camera_link" value="0.05" /> <!-- Size of square 'camera' box -->
-  <xacro:property name="axel_offset" value="0" /> <!-- Space btw top of beam and the each joint -->
+  <xacro:property name="camera_offsetX" value="-0.42" />
+  <xacro:property name="camera_offsetY" value="-0.20" />
+  <xacro:property name="camera_offsetZ" value="0.431" />
+  <xacro:property name="axel_offset" value="0" />
+  <xacro:property name="axel_offset" value="0" />
   <xacro:macro name="default_inertial" params="mass">
     <inertial>
@@ -65,5 +75,5 @@
     <child link="link1"/>
     <origin xyz="0 0 ${height0}" rpy="0 0 0"/>
-    <limit lower="${MinAngle}" upper="${MaxAngle}" effort="0" velocity="0"/>
+    <limit lower="${LowerLim_roll}" upper="${UpperLim_roll}" effort="0" velocity="0"/>
     <axis xyz="0 0 1"/>
     <dynamics damping="${damp_value}"/>
@@ -97,5 +107,5 @@
     <child link="link2"/>
     <origin xyz="0 0 ${height1 - axel_offset}" rpy="${radian} 0 0"/>
-    <limit lower="${MinAngle}" upper="${MaxAngle}" effort="0" velocity="0"/>
+    <limit lower="${LowerLim_joint1}" upper="${UpperLim_joint1}" effort="0" velocity="0"/>
     <axis xyz="0 0 1"/>
     <dynamics damping="${damp_value}"/>
@@ -129,5 +139,5 @@
     <child link="link3"/>
     <origin xyz="0 ${height2 - axel_offset*2} 0" rpy="${-radian} 0 0"/>
-    <limit lower="${MinAngle}" upper="${MaxAngle}" effort="0" velocity="0"/>
+    <limit lower="${LowerLim_roll}" upper="${UpperLim_roll}" effort="0" velocity="0"/>
     <axis xyz="0 0 1"/>
     <dynamics damping="${damp_value}"/>
@@ -161,5 +171,5 @@
     <child link="link4"/>
     <origin xyz="0 0 ${height3 - axel_offset*2}" rpy="${radian} 0 ${PI}"/>
-    <limit lower="${MinAngle}" upper="${MaxAngle}" effort="0" velocity="0"/>
+    <limit lower="${LowerLim_joint3}" upper="${UpperLim_joint3}" effort="0" velocity="0"/>
     <axis xyz="0 0 1"/>
     <dynamics damping="${damp_value}"/>
@@ -193,5 +203,5 @@
     <child link="link5"/>
     <origin xyz="0 ${height4 - axel_offset*2} 0" rpy="${-radian} 0 0"/>
-    <limit lower="${MinAngle}" upper="${MaxAngle}" effort="0" velocity="0"/>
+    <limit lower="${LowerLim_roll}" upper="${UpperLim_roll}" effort="0" velocity="0"/>
     <axis xyz="0 0 1"/>
     <dynamics damping="${damp_value}"/>
@@ -225,5 +235,5 @@
     <child link="link6"/>
     <origin xyz="0 0 ${height5 - axel_offset}" rpy="${radian} 0 0"/>
-    <limit lower="${MinAngle}" upper="${MaxAngle}" effort="0" velocity="0"/>
+    <limit lower="${LowerLim_joint5}" upper="${UpperLim_joint5}" effort="0" velocity="0"/>
     <axis xyz="0 0 1"/>
     <dynamics damping="${damp_value}"/>
@@ -283,18 +293,17 @@
   </link>
   <!-- End Effector -->
-  <xacro:macro name="gripper" params="prefix reflect">
+  <!-- diagnal settting -->
+  <!-- <xacro:macro name="gripper" params="prefix reflect">
     <joint name="${prefix}_gripper_joint" type="revolute">
       <axis xyz="0 ${reflect} 0"/>
-      <!-- <limit effort="1000.0" lower="-0.548" upper="0.548" velocity="0.5"/> -->
-      <limit lower="${MinAngle}" upper="${MaxAngle}" effort="0" velocity="0"/>
-      <origin rpy="0 0 0" xyz="${reflect*-0.01} 0 ${heightEEF}"/>
+      <limit lower="${LowerLim_roll}" upper="${UpperLim_roll}" effort="0" velocity="0"/>
+      <origin rpy="0 0 ${PI}" xyz="${reflect*-0.03} 0 ${heightEEF}"/>
       <parent link="EEFlink"/>
       <child link="${prefix}_gripper"/>
-      <limit effort="30" velocity="1.0"/>
       <dynamics damping="${damp_value}" friction="0.0"/>
     </joint>
     <link name="${prefix}_gripper">
       <visual>
-        <origin rpy="${(reflect-1)/2*pi} ${-radian} ${radian}" xyz="0 0 0"/>
+        <origin rpy="${(reflect-1)/2*pi} ${-radian} ${radian-PI}" xyz="0 0 0"/>
         <geometry>
           <mesh filename="package://urdf_tutorial/meshes/l_finger.dae"/>
@@ -305,5 +314,40 @@
           <mesh filename="package://urdf_tutorial/meshes/l_finger.dae"/>
         </geometry>
-        <origin rpy="${(reflect-1)/2*pi} ${-radian} ${radian}" xyz="0 0 0"/>
+        <origin rpy="${(reflect-1)/2*pi} ${-radian} ${radian-PI}" xyz="0 0 0"/>
+      </collision>
+      <xacro:default_inertial mass="0.05"/>
+    </link>
+    <transmission name="${prefix}_gripper_trans" type="SimpleTransmission">
+      <type>transmission_interface/SimpleTransmission</type>
+      <actuator name="${prefix}_gripper_motor">
+        <mechanicalReduction>1</mechanicalReduction>
+      </actuator>
+      <joint name="${prefix}_gripper_joint">
+        <hardwareInterface>PositionJointInterface</hardwareInterface>
+      </joint>
+    </transmission>
+  </xacro:macro> -->
+  <!--  pararell setting-->
+  <xacro:macro name="gripper" params="prefix reflect">
+    <joint name="${prefix}_gripper_joint" type="revolute">
+      <axis xyz="0 ${reflect} 0"/>
+      <limit lower="${LowerLim_roll}" upper="${UpperLim_roll}" effort="0" velocity="0"/>
+      <origin rpy="0 0 ${PI/2}" xyz="0 ${reflect*0.03} ${heightEEF}"/>
+      <parent link="EEFlink"/>
+      <child link="${prefix}_gripper"/>
+      <dynamics damping="${damp_value}" friction="0.0"/>
+    </joint>
+    <link name="${prefix}_gripper">
+      <visual>
+        <origin rpy="${(reflect-1)/2*pi} ${-radian} ${radian-PI}" xyz="0 0 0"/>
+        <geometry>
+          <mesh filename="package://urdf_tutorial/meshes/l_finger.dae"/>
+        </geometry>
+      </visual>
+      <collision>
+        <geometry>
+          <mesh filename="package://urdf_tutorial/meshes/l_finger.dae"/>
+        </geometry>
+        <origin rpy="${(reflect-1)/2*pi} ${-radian} ${radian-PI}" xyz="0 0 0"/>
       </collision>
       <xacro:default_inertial mass="0.05"/>
@@ -321,3 +365,43 @@
   <xacro:gripper prefix="left" reflect="1" />
   <xacro:gripper prefix="right" reflect="-1" />
+  <joint name="camerabase_joint" type="fixed">
+    <parent link="world"/>
+    <child link="D435base_link"/>
+    <origin xyz="${camera_offsetX} ${camera_offsetY} 0" rpy="0 0 0"/>
+  </joint>
+  <link name="D435base_link">
+    <collision>
+      <origin xyz="0 0 ${(camera_offsetZ-0.012)/2}" rpy="0 0 0"/>
+      <geometry>
+  <cylinder length="${camera_offsetZ-0.012}" radius="0.01"/>
+      </geometry>
+    </collision>
+    <visual>
+      <origin xyz="0 0 ${(camera_offsetZ-0.012)/2}" rpy="0 0 0"/>
+      <geometry>
+  <cylinder length="${camera_offsetZ-0.012}" radius="0.02"/>
+      </geometry>
+      <material name="black"/>
+    </visual>
+  </link>
+  <joint name="D435joint" type="fixed">
+    <parent link="D435base_link"/>
+    <child link="D435_link"/>
+    <origin xyz="0 0 ${camera_offsetZ}" rpy="${PI/2} 0 ${PI/2}"/>
+  </joint>
+  <link name="D435_link">
+    <visual>
+      <origin rpy="0 0 0" xyz="0 0 0.012"/>
+      <geometry>
+        <mesh filename="package://realsense2_description/meshes/d435.dae"/>
+      </geometry>
+    </visual>
+    <collision>
+      <geometry>
+        <mesh filename="package://realsense2_description/meshes/d435.dae"/>
+      </geometry>
+      <origin rpy="0 0 0" xyz="0 0 0.012"/>
+    </collision>
+    <xacro:default_inertial mass="0.05"/>
+  </link>
 </robot>

Commit message: create 2arm xacro

File: gazebo_ros_demos/rrbot_description/urdf/rrbot.xacro (robot description, xacro)
@@ -26,6 +26,7 @@
   <xacro:property name="heightEEF" value="0.03" /> <!-- Link 7  EEF Link-->
   <xacro:property name="damp_value"  value="0.0" /> <!-- Link 6 -->
+ <!--  camera reference from link0-->
   <xacro:property name="camera_offsetX" value="-0.42" />
-  <xacro:property name="camera_offsetY" value="-0.20" />
+  <xacro:property name="camera_offsetY" value="-0.182" />
   <xacro:property name="camera_offsetZ" value="0.431" />
   <xacro:property name="axel_offset" value="0" />
