Commit message: calc ik using trac-ik python

File: gazebo_ros_demos/rrbot_description/urdf/conbeL.xacro (robot description, xacro)
@@ -43,5 +43,5 @@
   <!-- ****************************************************************************** -->
   <xacro:joint_link_macro
-    prefix="" joint_name="fixed" joint_type="fixed" LowerLim="None" UpperLim="None"
+    prefix="L" joint_name="fixed" joint_type="fixed" LowerLim="None" UpperLim="None"
     parent="world" child="link0"
     width="${width}" height="${height0}" color="black" mass="1.0"
@@ -49,5 +49,5 @@
     Lx="0" Ly="0" Lz="${height0/2}" Lroll="0" Lpitch="0" Lyaw="0" />
   <xacro:joint_link_macro
-    prefix="" joint_name="joint0" joint_type="revolute" LowerLim="${LowerLim_roll}" UpperLim="${UpperLim_roll}"
+    prefix="L" joint_name="joint0" joint_type="revolute" LowerLim="${LowerLim_roll}" UpperLim="${UpperLim_roll}"
     parent="link0" child="link1"
     width="${width}" height="${height1}" color="orange" mass="1.0"
@@ -55,5 +55,5 @@
     Lx="0" Ly="0" Lz="${height1/2}" Lroll="0" Lpitch="0" Lyaw="0" />
   <xacro:joint_link_macro
-    prefix="" joint_name="joint1" joint_type="revolute" LowerLim="${LowerLim_joint1}" UpperLim="${UpperLim_joint1}"
+    prefix="L" joint_name="joint1" joint_type="revolute" LowerLim="${LowerLim_joint1}" UpperLim="${UpperLim_joint1}"
     parent="link1" child="link2"
     width="${width}" height="${height2}" color="black" mass="1.0"
@@ -61,5 +61,5 @@
     Lx="0" Ly="${height2/2}" Lz="0" Lroll="${PI/2}" Lpitch="0" Lyaw="0" />
   <xacro:joint_link_macro
-    prefix="" joint_name="joint2" joint_type="revolute" LowerLim="${LowerLim_roll}" UpperLim="${UpperLim_roll}"
+    prefix="L" joint_name="joint2" joint_type="revolute" LowerLim="${LowerLim_roll}" UpperLim="${UpperLim_roll}"
     parent="link2" child="link3"
     width="${width}" height="${height3}" color="orange" mass="1.0"
@@ -67,5 +67,5 @@
     Lx="0" Ly="0" Lz="${height3/2}" Lroll="0" Lpitch="0" Lyaw="0" />
   <xacro:joint_link_macro
-    prefix="" joint_name="joint3" joint_type="revolute" LowerLim="${LowerLim_joint3}" UpperLim="${UpperLim_joint3}"
+    prefix="L" joint_name="joint3" joint_type="revolute" LowerLim="${LowerLim_joint3}" UpperLim="${UpperLim_joint3}"
     parent="link3" child="link4"
     width="${width}" height="${height4}" color="black" mass="1.0"
@@ -73,5 +73,5 @@
     Lx="0" Ly="${height4/2}" Lz="0" Lroll="${-PI/2}" Lpitch="0" Lyaw="0" />
   <xacro:joint_link_macro
-    prefix="" joint_name="joint4" joint_type="revolute" LowerLim="${LowerLim_roll}" UpperLim="${UpperLim_roll}"
+    prefix="L" joint_name="joint4" joint_type="revolute" LowerLim="${LowerLim_roll}" UpperLim="${UpperLim_roll}"
     parent="link4" child="link5"
     width="${width}" height="${height5}" color="orange" mass="1.0"
@@ -79,5 +79,5 @@
     Lx="0" Ly="0" Lz="${height5/2}" Lroll="0" Lpitch="0" Lyaw="0" />
   <xacro:joint_link_macro
-    prefix="" joint_name="joint5" joint_type="revolute" LowerLim="${LowerLim_joint5}" UpperLim="${UpperLim_joint5}"
+    prefix="L" joint_name="joint5" joint_type="revolute" LowerLim="${LowerLim_joint5}" UpperLim="${UpperLim_joint5}"
     parent="link5" child="link6"
     width="${width}" height="${height6}" color="black" mass="1.0"
@@ -85,11 +85,11 @@
     Lx="0" Ly="${height6/2}" Lz="0" Lroll="${-PI/2}" Lpitch="0" Lyaw="0" />
   <xacro:joint_link_macro
-    prefix="" joint_name="EEFjoint" joint_type="fixed" LowerLim="None" UpperLim="None"
+    prefix="L" joint_name="EEFjoint" joint_type="fixed" LowerLim="None" UpperLim="None"
     parent="link6" child="EEFlink"
     width="${width}" height="${heightEEF}" color="red" mass="1.0"
     Jx="0" Jy="${height6}" Jz="0" Jroll="${-PI/2}" Jpitch="0" Jyaw="0"
     Lx="0" Ly="0" Lz="${heightEEF/2}" Lroll="0" Lpitch="0" Lyaw="0" />
-  <xacro:gripper prefix="" parent="EEFlink" parent_height="${heightEEF}" LorR="left" reflect="1" LowerLim_roll="${LowerLim_roll}"  UpperLim_roll="${UpperLim_roll}" PI="${PI}"/>
-  <xacro:gripper prefix="" parent="EEFlink" parent_height="${heightEEF}" LorR="right" reflect="-1" LowerLim_roll="${LowerLim_roll}"  UpperLim_roll="${UpperLim_roll}" PI="${PI}"/>
+  <xacro:gripper prefix="L" parent="EEFlink" parent_height="${heightEEF}" LorR="left" reflect="1" LowerLim_roll="${LowerLim_roll}"  UpperLim_roll="${UpperLim_roll}" PI="${PI}"/>
+  <xacro:gripper prefix="L" parent="EEFlink" parent_height="${heightEEF}" LorR="right" reflect="-1" LowerLim_roll="${LowerLim_roll}"  UpperLim_roll="${UpperLim_roll}" PI="${PI}"/>
   <!-- ****************************************************************************** -->
   <!--  RIGHT ARM DESCRIPTION -->

File: gazebo_ros_demos/rrbot_description/urdf/conbeR.xacro (robot description, xacro)
@@ -16,9 +16,9 @@
   <!-- upper limit of the angle -->
   <xacro:property name="UpperLim_roll"  value="2.617" />
-  <xacro:property name="UpperLim_joint1"  value="1.46239" />
+  <xacro:property name="UpperLim_joint1"  value="2.00644" />
   <xacro:property name="UpperLim_joint3"  value="2.26006" />
   <xacro:property name="UpperLim_joint5"  value="1.958382" />
   <xacro:property name="LowerLim_roll"  value= "-2.617" />
-  <xacro:property name="LowerLim_joint1"  value="-1.8816" />
+  <xacro:property name="LowerLim_joint1"  value="-1.8699" />
   <xacro:property name="LowerLim_joint3"  value="-1.7385" />
   <xacro:property name="LowerLim_joint5"  value="-1.677152" />
@@ -42,5 +42,5 @@
   <!--  LEFT ARM DESCRIPTION -->
   <!-- ****************************************************************************** -->
-  <xacro:joint_link_macro
+  <!-- <xacro:joint_link_macro
     prefix="" joint_name="fixed" joint_type="fixed" LowerLim="None" UpperLim="None"
     parent="world" child="link0"
@@ -91,9 +91,9 @@
     Lx="0" Ly="0" Lz="${heightEEF/2}" Lroll="0" Lpitch="0" Lyaw="0" />
   <xacro:gripper prefix="" parent="EEFlink" parent_height="${heightEEF}" LorR="left" reflect="1" LowerLim_roll="${LowerLim_roll}"  UpperLim_roll="${UpperLim_roll}" PI="${PI}"/>
-  <xacro:gripper prefix="" parent="EEFlink" parent_height="${heightEEF}" LorR="right" reflect="-1" LowerLim_roll="${LowerLim_roll}"  UpperLim_roll="${UpperLim_roll}" PI="${PI}"/>
+  <xacro:gripper prefix="" parent="EEFlink" parent_height="${heightEEF}" LorR="right" reflect="-1" LowerLim_roll="${LowerLim_roll}"  UpperLim_roll="${UpperLim_roll}" PI="${PI}"/> -->
   <!-- ****************************************************************************** -->
   <!--  RIGHT ARM DESCRIPTION -->
   <!-- ****************************************************************************** -->
-  <!-- <xacro:joint_link_macro
+  <xacro:joint_link_macro
     prefix="R" joint_name="fixed" joint_type="fixed" LowerLim="None" UpperLim="None"
     parent="world" child="link0"
@@ -144,5 +144,5 @@
     Lx="0" Ly="0" Lz="${heightEEF/2}" Lroll="0" Lpitch="0" Lyaw="0" />
   <xacro:gripper prefix="R" parent="EEFlink" parent_height="${heightEEF}" LorR="left" reflect="1" LowerLim_roll="${LowerLim_roll}"  UpperLim_roll="${UpperLim_roll}" PI="${PI}"/>
-  <xacro:gripper prefix="R" parent="EEFlink" parent_height="${heightEEF}" LorR="Right" reflect="-1" LowerLim_roll="${LowerLim_roll}"  UpperLim_roll="${UpperLim_roll}" PI="${PI}"/> -->
+  <xacro:gripper prefix="R" parent="EEFlink" parent_height="${heightEEF}" LorR="right" reflect="-1" LowerLim_roll="${LowerLim_roll}"  UpperLim_roll="${UpperLim_roll}" PI="${PI}"/>
   <!-- ****************************************************************************** -->
   <!--  D435 DESCRIPTION -->

Commit message: made arm script indivizually

File: gazebo_ros_demos/rrbot_description/urdf/conbeL.xacro (robot description, xacro)
@@ -16,9 +16,11 @@
   <!-- upper limit of the angle -->
   <xacro:property name="UpperLim_roll"  value="2.617" />
-  <xacro:property name="UpperLim_joint1"  value="1.46239" />
+  <!-- <xacro:property name="UpperLim_joint1"  value="1.46239" />  for DX-->
+  <xacro:property name="UpperLim_joint1"  value="2.00644" />
   <xacro:property name="UpperLim_joint3"  value="2.26006" />
   <xacro:property name="UpperLim_joint5"  value="1.958382" />
   <xacro:property name="LowerLim_roll"  value= "-2.617" />
-  <xacro:property name="LowerLim_joint1"  value="-1.8816" />
+  <!-- <xacro:property name="LowerLim_joint1"  value="-1.8816" />  for DX-->
+  <xacro:property name="LowerLim_joint1"  value="-1.8699" />
   <xacro:property name="LowerLim_joint3"  value="-1.7385" />
   <xacro:property name="LowerLim_joint5"  value="-1.677152" />

Commit message: update dolly&jog

File: gazebo_ros_demos/rrbot_description/urdf/conbeL.xacro (robot description, xacro)
@@ -7,5 +7,5 @@
   <xacro:property name="width"     value="0.05" /> <!-- Square dimensions (widthxwidth) of beams -->
   <xacro:property name="height0"   value="0.275" /> <!-- Link 0 -->
-  <xacro:property name="height1"   value="0.036" /> <!-- Link 1 -->
+  <xacro:property name="height1"   value="0.050" /> <!-- Link 1 -->
   <xacro:property name="height2"   value="0.105" /> <!-- Link 2 -->
   <xacro:property name="height3"   value="0.043" /> <!-- Link 3 -->
@@ -16,9 +16,11 @@
   <!-- upper limit of the angle -->
   <xacro:property name="UpperLim_roll"  value="2.617" />
+  <xacro:property name="UpperLim_roll_joint0"  value="0.86" />
   <!-- <xacro:property name="UpperLim_joint1"  value="1.46239" />  for DX-->
   <xacro:property name="UpperLim_joint1"  value="2.00644" />
-  <xacro:property name="UpperLim_joint3"  value="2.26006" />
+  <xacro:property name="UpperLim_joint3"  value="2.18" />
   <xacro:property name="UpperLim_joint5"  value="1.958382" />
   <xacro:property name="LowerLim_roll"  value= "-2.617" />
+  <xacro:property name="LowerLim_roll_joint0"  value= "-1.87" />
   <!-- <xacro:property name="LowerLim_joint1"  value="-1.8816" />  for DX-->
   <xacro:property name="LowerLim_joint1"  value="-1.8699" />
@@ -51,5 +53,5 @@
     Lx="0" Ly="0" Lz="${height0/2}" Lroll="0" Lpitch="0" Lyaw="0" />
   <xacro:joint_link_macro
-    prefix="L" joint_name="joint0" joint_type="revolute" LowerLim="${LowerLim_roll}" UpperLim="${UpperLim_roll}"
+    prefix="L" joint_name="joint0" joint_type="revolute" LowerLim="${LowerLim_roll_joint0}" UpperLim="${UpperLim_roll_joint0}"
     parent="link0" child="link1"
     width="${width}" height="${height1}" color="orange" mass="1.0"

File: gazebo_ros_demos/rrbot_description/urdf/conbeR.xacro (robot description, xacro)
@@ -7,5 +7,5 @@
   <xacro:property name="width"     value="0.05" /> <!-- Square dimensions (widthxwidth) of beams -->
   <xacro:property name="height0"   value="0.275" /> <!-- Link 0 -->
-  <xacro:property name="height1"   value="0.036" /> <!-- Link 1 -->
+  <xacro:property name="height1"   value="0.050" /> <!-- Link 1 -->
   <xacro:property name="height2"   value="0.105" /> <!-- Link 2 -->
   <xacro:property name="height3"   value="0.043" /> <!-- Link 3 -->
@@ -16,8 +16,10 @@
   <!-- upper limit of the angle -->
   <xacro:property name="UpperLim_roll"  value="2.617" />
+  <xacro:property name="UpperLim_roll_joint0"  value="0.86" />
   <xacro:property name="UpperLim_joint1"  value="2.00644" />
-  <xacro:property name="UpperLim_joint3"  value="2.26006" />
+  <xacro:property name="UpperLim_joint3"  value="2.18" />
   <xacro:property name="UpperLim_joint5"  value="1.958382" />
   <xacro:property name="LowerLim_roll"  value= "-2.617" />
+  <xacro:property name="LowerLim_roll_joint0"  value= "-1.87" />
   <xacro:property name="LowerLim_joint1"  value="-1.8699" />
   <xacro:property name="LowerLim_joint3"  value="-1.7385" />
@@ -40,57 +42,4 @@
   <link name="world"/>
   <!-- ****************************************************************************** -->
-  <!--  LEFT ARM DESCRIPTION -->
-  <!-- ****************************************************************************** -->
-  <!-- <xacro:joint_link_macro
-    prefix="" joint_name="fixed" joint_type="fixed" LowerLim="None" UpperLim="None"
-    parent="world" child="link0"
-    width="${width}" height="${height0}" color="black" mass="1.0"
-    Jx="0" Jy="0" Jz="0" Jroll="0" Jpitch="0" Jyaw="0"
-    Lx="0" Ly="0" Lz="${height0/2}" Lroll="0" Lpitch="0" Lyaw="0" />
-  <xacro:joint_link_macro
-    prefix="" joint_name="joint0" joint_type="revolute" LowerLim="${LowerLim_roll}" UpperLim="${UpperLim_roll}"
-    parent="link0" child="link1"
-    width="${width}" height="${height1}" color="orange" mass="1.0"
-    Jx="0" Jy="0" Jz="${height0}" Jroll="0" Jpitch="0" Jyaw="0"
-    Lx="0" Ly="0" Lz="${height1/2}" Lroll="0" Lpitch="0" Lyaw="0" />
-  <xacro:joint_link_macro
-    prefix="" joint_name="joint1" joint_type="revolute" LowerLim="${LowerLim_joint1}" UpperLim="${UpperLim_joint1}"
-    parent="link1" child="link2"
-    width="${width}" height="${height2}" color="black" mass="1.0"
-    Jx="0" Jy="0" Jz="${height1}" Jroll="${PI/2}" Jpitch="0" Jyaw="0"
-    Lx="0" Ly="${height2/2}" Lz="0" Lroll="${PI/2}" Lpitch="0" Lyaw="0" />
-  <xacro:joint_link_macro
-    prefix="" joint_name="joint2" joint_type="revolute" LowerLim="${LowerLim_roll}" UpperLim="${UpperLim_roll}"
-    parent="link2" child="link3"
-    width="${width}" height="${height3}" color="orange" mass="1.0"
-    Jx="0" Jy="${height2}" Jz="0" Jroll="${-PI/2}" Jpitch="0" Jyaw="0"
-    Lx="0" Ly="0" Lz="${height3/2}" Lroll="0" Lpitch="0" Lyaw="0" />
-  <xacro:joint_link_macro
-    prefix="" joint_name="joint3" joint_type="revolute" LowerLim="${LowerLim_joint3}" UpperLim="${UpperLim_joint3}"
-    parent="link3" child="link4"
-    width="${width}" height="${height4}" color="black" mass="1.0"
-    Jx="0" Jy="0" Jz="${height3}" Jroll="${PI/2}" Jpitch="0" Jyaw="${PI}"
-    Lx="0" Ly="${height4/2}" Lz="0" Lroll="${-PI/2}" Lpitch="0" Lyaw="0" />
-  <xacro:joint_link_macro
-    prefix="" joint_name="joint4" joint_type="revolute" LowerLim="${LowerLim_roll}" UpperLim="${UpperLim_roll}"
-    parent="link4" child="link5"
-    width="${width}" height="${height5}" color="orange" mass="1.0"
-    Jx="0" Jy="${height4}" Jz="0" Jroll="${-PI/2}" Jpitch="0" Jyaw="0"
-    Lx="0" Ly="0" Lz="${height5/2}" Lroll="0" Lpitch="0" Lyaw="0" />
-  <xacro:joint_link_macro
-    prefix="" joint_name="joint5" joint_type="revolute" LowerLim="${LowerLim_joint5}" UpperLim="${UpperLim_joint5}"
-    parent="link5" child="link6"
-    width="${width}" height="${height6}" color="black" mass="1.0"
-    Jx="0" Jy="0" Jz="${height5}" Jroll="${PI/2}" Jpitch="0" Jyaw="0"
-    Lx="0" Ly="${height6/2}" Lz="0" Lroll="${-PI/2}" Lpitch="0" Lyaw="0" />
-  <xacro:joint_link_macro
-    prefix="" joint_name="EEFjoint" joint_type="fixed" LowerLim="None" UpperLim="None"
-    parent="link6" child="EEFlink"
-    width="${width}" height="${heightEEF}" color="red" mass="1.0"
-    Jx="0" Jy="${height6}" Jz="0" Jroll="${-PI/2}" Jpitch="0" Jyaw="0"
-    Lx="0" Ly="0" Lz="${heightEEF/2}" Lroll="0" Lpitch="0" Lyaw="0" />
-  <xacro:gripper prefix="" parent="EEFlink" parent_height="${heightEEF}" LorR="left" reflect="1" LowerLim_roll="${LowerLim_roll}"  UpperLim_roll="${UpperLim_roll}" PI="${PI}"/>
-  <xacro:gripper prefix="" parent="EEFlink" parent_height="${heightEEF}" LorR="right" reflect="-1" LowerLim_roll="${LowerLim_roll}"  UpperLim_roll="${UpperLim_roll}" PI="${PI}"/> -->
-  <!-- ****************************************************************************** -->
   <!--  RIGHT ARM DESCRIPTION -->
   <!-- ****************************************************************************** -->
@@ -102,5 +51,5 @@
     Lx="0" Ly="0" Lz="${height0/2}" Lroll="0" Lpitch="0" Lyaw="0" />
   <xacro:joint_link_macro
-    prefix="R" joint_name="joint0" joint_type="revolute" LowerLim="${LowerLim_roll}" UpperLim="${UpperLim_roll}"
+    prefix="R" joint_name="joint0" joint_type="revolute" LowerLim="${LowerLim_roll_joint0}" UpperLim="${UpperLim_roll_joint0}"
     parent="link0" child="link1"
     width="${width}" height="${height1}" color="orange" mass="1.0"

Commit message: 1d bofore comp

File: gazebo_ros_demos/rrbot_description/urdf/conbeL.xacro (robot description, xacro)
@@ -12,6 +12,8 @@
   <xacro:property name="height4"   value="0.041" /> <!-- Link 4 -->
   <xacro:property name="height5"   value="0.11" /> <!-- Link 5 -->
-  <xacro:property name="height6"   value="0.125" /> <!-- Link 6 -->
-  <xacro:property name="heightEEF" value="0.03" /> <!-- Link 7  EEF Link-->
+  <!-- Link 6 -->
+  <!-- <xacro:property name="height6"   value="0.125" />  -->
+  <xacro:property name="height6"   value="0.145" /> <!-- Link 6 -->
+  <xacro:property name="heightEEF" value="0.01" /> <!-- Link 7  EEF Link 3=>5-->
   <!-- upper limit of the angle -->
   <xacro:property name="UpperLim_roll"  value="2.617" />

File: gazebo_ros_demos/rrbot_description/urdf/conbeR.xacro (robot description, xacro)
@@ -13,5 +13,5 @@
   <xacro:property name="height5"   value="0.11" /> <!-- Link 5 -->
   <xacro:property name="height6"   value="0.125" /> <!-- Link 6 -->
-  <xacro:property name="heightEEF" value="0.03" /> <!-- Link 7  EEF Link-->
+  <xacro:property name="heightEEF" value="0.10" /> <!-- Link 7  EEF Link 3=> 5-->
   <!-- upper limit of the angle -->
   <xacro:property name="UpperLim_roll"  value="2.617" />
